Commit message: Fixed lanuch files.

File: snailbot_description/urdf/snailbot.urdf (robot description, URDF)
Before this commit: robot snailbot, 2 links, 1 joints
Links:
- link base_link: geometry visual mesh filename=package://snailbot_description/meshes/snailbot.stl scale=0.001 0.001 0.001

Commit message: Added some launch files for navigation.  Also, updated URDF.

File: snailbot_description/urdf/snailbot.urdf (robot description, URDF)
Before this commit: robot snailbot, 2 links, 1 joints
Links:
- added link camera_link; visual mesh filename=package://snailbot_description/meshes/xtion.stl
Joints:
- added joint camera_joint: type fixed, parent base_link, child camera_link, origin xyz=0 0 0 rpy=0 0 0

Commit message: Updated xtion position in URDF.

File: snailbot_description/urdf/snailbot.urdf (robot description, URDF)
Before this commit: robot snailbot, 3 links, 2 joints
Joints:
- joint camera_joint: origin xyz=0 0 0 rpy=0 0 0 -> xyz=0.125 0 0 rpy=0 0 0

Commit message: Updated URDF.

File: snailbot_description/urdf/snailbot.urdf (robot description, URDF)
Before this commit: robot snailbot, 3 links, 2 joints
Joints:
- joint base_footprint_joint: origin xyz=0 0 0 rpy=0 0 0 -> xyz=0 0 0.04 rpy=0 0 0
- joint camera_joint: origin xyz=0.125 0 0 rpy=0 0 0 -> xyz=0.125 0 0.15 rpy=0 0 0

Commit message: Minor updates to URDF.

File: snailbot_description/urdf/snailbot.urdf (robot description, URDF)
Before this commit: robot snailbot, 3 links, 2 joints
Links:
- removed link base_footprint
Joints:
- removed joint base_footprint_joint
- joint camera_joint: origin xyz=0.125 0 0.15 rpy=0 0 0 -> xyz=0.095 0 0.105 rpy=0 0 0
